File: Hardware/SAMD21_Pro_RF.brd (EAGLE design)
At the start: 44.5 x 30.5 mm, 129 parts, among them J12 JST, J13 U.FL, J7 PTH, J9 External On/Off, Q1 2.5A/30V, U1 MCP73831, U3 RFM95W, U4 ATSAMD21G, U6 3.3V, Y1 32.768kHz

Commit message: Gerbers
Parts:
- moved U$25 0.25 mm to (22.4, 10.3)
- moved U$35 0.25 mm to (18.9, 10.3)
- moved FD1 0.13 mm to (1.27, 3.94)
- moved FD3 0.13 mm to (1.27, 3.94)
Routing:
- net STAT_LED: track 28.3 -> 29.2 mm
- net N$17: track 23.8 -> 23.2 mm
- net TXO: track 21.1 -> 21.7 mm
