File: Production/SAMD21_Pro_RF-Panel.brd (EAGLE design)
At the start: 164.6 x 106.2 mm, 1248 parts, among them J100 PTH, J102 External On/Off, J106 JST, J110 U.FL, J114 PTH, J116 External On/Off, J12 JST, J120 JST, J124 U.FL, J13 U.FL, J16 PTH, J18 External On/Off, J22 JST, J26 U.FL, J30 PTH, J32 External On/Off, J36 JST, J40 U.FL, J44 PTH, J46 External On/Off, J50 JST, J54 U.FL, J58 PTH, J60 External On/Off, J64 JST, J68 U.FL, J7 PTH, J72 PTH, J74 External On/Off, J78 JST, J82 U.FL, J86 PTH, J88 External On/Off, J9 External On/Off, J92 JST, J96 U.FL, Q1 2.5A/30V, Q2 2.5A/30V, Q3 2.5A/30V, Q4 2.5A/30V, Q5 2.5A/30V, Q6 2.5A/30V, Q7 2.5A/30V, Q8 2.5A/30V, Q9 2.5A/30V, U1 MCP73831, U10 3.3V, U11 ATSAMD21G, U12 RFM95W, U13 MCP73831, U14 3.3V, U15 ATSAMD21G, U16 RFM95W, U17 MCP73831, U18 3.3V, U19 ATSAMD21G, U2 MCP73831, U20 RFM95W, U21 MCP73831, U22 3.3V, U23 ATSAMD21G, U24 RFM95W, U25 MCP73831, U26 3.3V, U27 ATSAMD21G, U28 RFM95W, U29 MCP73831, U3 RFM95W, U30 3.3V, U31 ATSAMD21G, U32 RFM95W, U33 MCP73831, U34 3.3V, U35 ATSAMD21G, U36 RFM95W, U4 ATSAMD21G, U5 3.3V, U6 3.3V, U7 ATSAMD21G, U8 RFM95W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

Commit message: Updated panel fiducials
Parts:
- moved E$3 7.57 mm to (130.0, 94.6)
- moved E$4 7.57 mm to (130.0, 94.6)
Changed lines of the file:
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@@
 <element name="E$1" library="SparkFun-Aesthetics" package="FIDUCIAL-1X2" value="" x="9.398" y="94.5515" smashed="yes"/>
 <element name="E$2" library="SparkFun-Aesthetics" package="FIDUCIAL-1X2" value="" x="9.398" y="94.5515" smashed="yes" rot="MR0"/>
-<element name="E$3" library="SparkFun-Aesthetics" package="FIDUCIAL-1X2" value="" x="137.6045" y="94.5515" smashed="yes"/>
-<element name="E$4" library="SparkFun-Aesthetics" package="FIDUCIAL-1X2" value="" x="137.6045" y="94.5515" smashed="yes" rot="MR0"/>
+<element name="E$3" library="SparkFun-Aesthetics" package="FIDUCIAL-1X2" value="" x="130.0353" y="94.5515" smashed="yes"/>
+<element name="E$4" library="SparkFun-Aesthetics" package="FIDUCIAL-1X2" value="" x="130.0353" y="94.5515" smashed="yes" rot="MR0"/>
 <element name="E$5" library="SparkFun-Retired" package="FIDUCIAL-1.5X3" value="" x="9.398" y="-2.0955" smashed="yes"/>
 <element name="E$6" library="SparkFun-Retired" package="FIDUCIAL-1.5X3" value="" x="9.398" y="-2.0955" smashed="yes" rot="MR0"/>
